Commit message: changes joints' type to revolute and adds limits to joints (to be modified later)

File: control/ros_ws/src/controls/config/Robot.urdf (robot description, URDF)
Before this commit: robot /home/thomas-xavier/github/Alpha-Bear-Omega-3/control/ros_ws/src/alphabearomega3/worlds/Robot.urdf, 18 links, 17 joints
Joints:
- joint FL_femur_servo: limit effort=1000 velocity=50 -> lower=0 upper=${pi/2} effort=1000 velocity=50; type continuous -> revolute
- joint FL_shoulder_servo: limit effort=1000 velocity=50 -> lower=${-pi/3} upper=${pi/3} effort=1000 velocity=50; type continuous -> revolute
- joint FL_tibia_servo: limit effort=1000 velocity=50 -> lower=0 upper=${pi/2} effort=1000 velocity=50; type continuous -> revolute
- joint FR_femur_servo: limit effort=1000 velocity=50 -> lower=0 upper=${pi/2} effort=1000 velocity=50; type continuous -> revolute
- joint FR_shoulder_servo: limit effort=1000 velocity=50 -> lower=${-pi/3} upper=${pi/3} effort=1000 velocity=50; type continuous -> revolute
- joint FR_tibia_servo: limit effort=1000 velocity=50 -> lower=0 upper=${pi/2} effort=1000 velocity=50; type continuous -> revolute
- joint RL_femur_servo: limit effort=1000 velocity=50 -> lower=0 upper=${pi/2} effort=1000 velocity=50; type continuous -> revolute
- joint RL_shoulder_servo: limit effort=1000 velocity=50 -> lower=${-pi/3} upper=${pi/3} effort=1000 velocity=50; type continuous -> revolute
- joint RL_tibia_servo: limit effort=1000 velocity=50 -> lower=0 upper=${pi/2} effort=1000 velocity=50; type continuous -> revolute
- joint RR_femur_servo: limit effort=1000 velocity=50 -> lower=0 upper=${pi/2} effort=1000 velocity=50; type continuous -> revolute
- joint RR_shoulder_servo: limit effort=1000 velocity=50 -> lower=${-pi/3} upper=${pi/3} effort=1000 velocity=50; type continuous -> revolute
- joint RR_tibia_servo: limit effort=1000 velocity=50 -> lower=0 upper=${pi/2} effort=1000 velocity=50; type continuous -> revolute
