Commit message: Changement de parametres pour la marche

File: control/ros_ws/src/alphabearomega3/worlds/Robot.urdf (robot description, URDF)
Before this commit: robot /home/thomas-xavier/github/Alpha-Bear-Omega-3/control/ros_ws/src/alphabearomega3/worlds/Robot.urdf, 18 links, 17 joints
Links:
- link FL_tibia: geometry collision box size=0.025 0.025 0.18; visual box size=0.025 0.025 0.18
- link FR_tibia: geometry collision box size=0.025 0.025 0.18; visual box size=0.025 0.025 0.18
- link RL_tibia: geometry collision box size=0.025 0.025 0.18; visual box size=0.025 0.025 0.18
- link RR_tibia: geometry collision box size=0.025 0.025 0.18; visual box size=0.025 0.025 0.18
